File: Platine/HM-LC-Sw1-Pl-DN-R1_OBII.kicad_pcb (KiCad board)
At the start: 2 copper layers, 17.8 x 24 mm, 9 parts, among them J3 Conn_01x01_Female, U1 ATmega328P-AU, U2 CC1101, U3 WROOM-02-DUKOS

Commit message: Add files via upload
Routing:
- net VCC: track 13.3 -> 16.8 mm
Changed lines of the file:
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@@
     (thickness 1.6)
     (drawings 19)
-    (tracks 118)
+    (tracks 122)
     (zones 0)
     (modules 9)
@@
   (segment (start 141.7 99.375) (end 141.825 99.25) (width 0.25) (layer B.Cu) (net 22))
   (segment (start 141.7 101.25) (end 141.7 99.375) (width 0.25) (layer B.Cu) (net 22))
+  (segment (start 141.025001 101.924999) (end 141.025001 102.274999) (width 0.25) (layer F.Cu) (net 22))
+  (segment (start 141.025001 101.924999) (end 141.7 101.25) (width 0.25) (layer F.Cu) (net 22))
+  (segment (start 140.8 100.35) (end 141.7 101.25) (width 0.25) (layer F.Cu) (net 22))
+  (segment (start 141.7 101.25) (end 141.025001 100.574999) (width 0.25) (layer F.Cu) (net 22))
   (segment (start 153.6 97.75) (end 155.95 97.75) (width 0.25) (layer F.Cu) (net 24))
   (segment (start 153.6 97.75) (end 153.6 97.175) (width 0.25) (layer F.Cu) (net 24))
@@
     (min_thickness 0.254)
     (keepout (tracks allowed) (vias allowed) (copperpour not_allowed))
-    (fill (arc_segments 16) (thermal_gap 0.508) (thermal_bridge_width 0.508) (smoothing chamfer))
+    (fill (arc_segments 16) (thermal_gap 0.508) (thermal_bridge_width 0.508))
     (polygon
       (pts
@@
     (min_thickness 0.254)
     (keepout (tracks allowed) (vias allowed) (copperpour not_allowed))
-    (fill (arc_segments 16) (thermal_gap 0.508) (thermal_bridge_width 0.508) (smoothing chamfer))
+    (fill (arc_segments 16) (thermal_gap 0.508) (thermal_bridge_width 0.508))
     (polygon
       (pts
@@
     )
   )
-  (zone (net 0) (net_name "") (layers F&B.Cu) (hatch edge 0.508)
-    (connect_pads (clearance 0.508))
+  (zone (net 0) (net_name "") (layer B.Cu) (hatch edge 0.508)
+    (connect_pads (clearance 0.408))
     (min_thickness 0.254)
     (keepout (tracks allowed) (vias allowed) (copperpour not_allowed))
-    (fill (arc_segments 16) (thermal_gap 0.508) (thermal_bridge_width 0.508) (smoothing chamfer))
+    (fill (arc_segments 16) (thermal_gap 0.508) (thermal_bridge_width 0.508))
     (polygon
       (pts
-        (xy 142.4 100.3) (xy 142.4 100.1) (xy 142.7 100) (xy 143.3 100.3) (xy 143.3 100.4)
-        (xy 142.9 100.8) (xy 142.4 100.4)
+        (xy 143.1 101) (xy 142.4 100.6) (xy 142.4 100.1) (xy 142.7 100) (xy 143.3 100.4)
+        (xy 143.3 100.7)
       )
     )
